File: sdm27ev/sdm27ev-vcu/hardware/sdm27ev-vcu-v1/sdm27ev-vcu-v1.kicad_sch (KiCad schematic)
At the start: 30 parts, among them J1 6437288-1, J2 6437288-1, J4 2201778-1, SW1 SW_Push, SW2 SW_Push, SW3 SW_Push, U1 ESP32-P4-Core, U2 CH32V003JxMx

Commit message: added VCU digital input protection
Other:
- added sheet Digital IO (DigitalIO.kicad_sch)
Changed lines of the file:
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@@
+		)
+	)
+	(sheet
+		(at 12.7 160.02)
+		(size 16.51 35.56)
+		(exclude_from_sim no)
+		(in_bom yes)
+		(on_board yes)
+		(dnp no)
+		(fields_autoplaced yes)
+		(stroke
+			(width 0.1524)
+			(type solid)
+		)
+		(fill
+			(color 0 0 0 0)
+		)
+		(property "Sheetname" "Digital IO"
+			(at 12.7 159.3084 0)
+			(show_name no)
+			(do_not_autoplace no)
+			(effects
+				(font
+					(size 1.27 1.27)
+				)
+				(justify left bottom)
+			)
+		)
+		(property "Sheetfile" "DigitalIO.kicad_sch"
+			(at 12.7 196.1646 0)
+			(show_name no)
+			(do_not_autoplace no)
+			(effects
+				(font
+					(size 1.27 1.27)
+				)
+				(justify left top)
+			)
+		)
+		(instances
+			(project "sdm27ev-vcu-v1"
+				(path "/aaff56d4-6a2c-4b9b-8d6c-def2b75cacc9"
+					(page "5")
+				)
+			)
 		)
 	)
