File: sdm27ev/sdm27ev-vcu/hardware/sdm27ev-vcu-v1/sdm27ev-vcu-v1.kicad_pcb (KiCad board)
At the start: 2 copper layers, 92 x 60 mm, 4 parts, among them J1 6437288-1, J2 6437288-1

Commit message: EV VCU edits, mostly organizational and pre layout/footprint assigned
Parts:
- removed J1, J2: 6437288-1, SDM27 EV VCU:TE_6437288-1
- removed REF**: microSD_HC_Molex_104031-0811, SDM:microSD_HC_Molex_104031-0811
- removed REF**: USB_C_Receptacle_GCT_USB4105-xx-A_16P_TopMnt_Horizontal, Connector_USB:USB_C_Receptacle_GCT_USB4105-xx-A_16P_TopMnt_Horizontal
- added C1: 100nF, Capacitor_SMD:C_0603_1608Metric, F.Cu at (145.6, 71.3)
- added C10: 10uF, Capacitor_SMD:C_0603_1608Metric, F.Cu at (162.8, 70.4)
- added C100: 20.5nF, Capacitor_SMD:C_0603_1608Metric, F.Cu at (14.7, 44.9)
- added C101: 20.5nF, Capacitor_SMD:C_0603_1608Metric, F.Cu at (18.1, 44.9)
- added C102: 20.5nF, Capacitor_SMD:C_0603_1608Metric, F.Cu at (21.5, 44.9)
- added C103: 20.5nF, Capacitor_SMD:C_0603_1608Metric, F.Cu at (179.7, 35.3)
- added C104: 20.5nF, Capacitor_SMD:C_0603_1608Metric, F.Cu at (179.7, 37.9)
- added C105: 20.5nF, Capacitor_SMD:C_0603_1608Metric, F.Cu at (179.7, 40.4)
- added C106: 20.5nF, Capacitor_SMD:C_0603_1608Metric, F.Cu at (183.7, 12.8)
- added C107: 100nF, Capacitor_SMD:C_0603_1608Metric, F.Cu at (12.0, 37.8)
- added C11: 100nF, Capacitor_SMD:C_0603_1608Metric, F.Cu at (162.8, 72.9)
- added C12: 10nF, Capacitor_SMD:C_0603_1608Metric, F.Cu at (188.5, 51.7)
- added C13: 10uF, Capacitor_SMD:C_0805_2012Metric, F.Cu at (204.8, 51.9)
- added C14: 10uF, Capacitor_SMD:C_0805_2012Metric, F.Cu at (204.8, 54.9)
- added C15: 100nF, Capacitor_SMD:C_0603_1608Metric, F.Cu at (188.5, 54.2)
- added C16: 10uF, Capacitor_SMD:C_0805_2012Metric, F.Cu at (204.8, 57.9)
- added C17: 100nF, Capacitor_SMD:C_0603_1608Metric, F.Cu at (188.5, 56.7)
- added C18: 10uF, Capacitor_SMD:C_0805_2012Metric, F.Cu at (204.8, 60.9)
- added C19: 1uF, Capacitor_SMD:C_0603_1608Metric, F.Cu at (188.5, 59.2)
- added C2: 100nF, Capacitor_SMD:C_0603_1608Metric, F.Cu at (145.6, 73.8)
- added C20: 1uF, Capacitor_SMD:C_0603_1608Metric, F.Cu at (188.5, 61.7)
- added C21: 1uF, Capacitor_SMD:C_0603_1608Metric, F.Cu at (188.5, 64.2)
- added C22: 100nF, Capacitor_SMD:C_0603_1608Metric, F.Cu at (5.40, 39.3)
- added C23: 100nF, Capacitor_SMD:C_0603_1608Metric, F.Cu at (115.7, 48.7)
- added C24: 100nF, Capacitor_SMD:C_0603_1608Metric, F.Cu at (188.5, 66.7)
- added C25: 4.7uF, Capacitor_SMD:C_0805_2012Metric, F.Cu at (204.8, 64.0)
- added C26: 100nF, Capacitor_SMD:C_0603_1608Metric, F.Cu at (188.5, 69.2)
- added C27: 33pF, Capacitor_SMD:C_0603_1608Metric, F.Cu at (192.5, 51.7)
- added C28: 4.7uF, Capacitor_SMD:C_0805_2012Metric, F.Cu at (204.8, 67.0)
- added C29: 33uF, Capacitor_SMD:C_0805_2012Metric, F.Cu at (204.8, 70.0)
- added C3: 100nF, Capacitor_SMD:C_0603_1608Metric, F.Cu at (145.6, 76.3)
- added C30: 33uF, Capacitor_SMD:C_0805_2012Metric, F.Cu at (204.8, 73.0)
- added C31: 1uF, Capacitor_SMD:C_0603_1608Metric, F.Cu at (192.5, 54.2)
- added C32: 100nF, Capacitor_SMD:C_0603_1608Metric, F.Cu at (192.5, 56.7)
- added C33: 1uF, Capacitor_SMD:C_0603_1608Metric, F.Cu at (192.5, 59.2)
- added C34: 100nF, Capacitor_SMD:C_0603_1608Metric, F.Cu at (192.5, 61.7)
- added C35: 1uF, Capacitor_SMD:C_0603_1608Metric, F.Cu at (192.5, 64.2)
- added C36: 1uF, Capacitor_SMD:C_0603_1608Metric, F.Cu at (192.5, 66.7)
- added C37: 1uF, Capacitor_SMD:C_0603_1608Metric, F.Cu at (192.5, 69.2)
- added C38: 1uF, Capacitor_SMD:C_0603_1608Metric, F.Cu at (196.5, 51.7)
- added C39: 1uF, Capacitor_SMD:C_0603_1608Metric, F.Cu at (196.5, 54.2)
- added C4: 100nF, Capacitor_SMD:C_0603_1608Metric, F.Cu at (2.40, 39.4)
- added C5: 100nF, Capacitor_SMD:C_0603_1608Metric, F.Cu at (115.7, 51.7)
- added C6: 100nF, Capacitor_SMD:C_0603_1608Metric, F.Cu at (149.6, 73.8)
- added C7: 100nF, Capacitor_SMD:C_0603_1608Metric, F.Cu at (162.8, 65.4)
- added C8: 1uF, Capacitor_SMD:C_0603_1608Metric, F.Cu at (162.8, 67.9)
- added C82: 100nF, Capacitor_SMD:C_0603_1608Metric, F.Cu at (9.60, 36.6)
- added C83: 100nF, Capacitor_SMD:C_0603_1608Metric, F.Cu at (14.5, 36.6)
- added C84: 100nF, Capacitor_SMD:C_0603_1608Metric, F.Cu at (16.4, 36.6)
- added C85: 100nF, Capacitor_SMD:C_0603_1608Metric, F.Cu at (21.3, 36.6)
- added C86: 100nF, Capacitor_SMD:C_0603_1608Metric, F.Cu at (175.7, 22.8)
- added C87: 100nF, Capacitor_SMD:C_0603_1608Metric, F.Cu at (175.7, 25.3)
- added C88: 100nF, Capacitor_SMD:C_0603_1608Metric, F.Cu at (175.7, 27.8)
- added C89: 100nF, Capacitor_SMD:C_0603_1608Metric, F.Cu at (175.7, 30.3)
- added C90: 100nF, Capacitor_SMD:C_0603_1608Metric, F.Cu at (18.9, 37.8)
- added C91: 10n, Capacitor_SMD:C_0603_1608Metric, F.Cu at (10.3, 41.9)
- added C92: 10n, Capacitor_SMD:C_0603_1608Metric, F.Cu at (13.8, 41.9)
- added C93: 10n, Capacitor_SMD:C_0603_1608Metric, F.Cu at (17.4, 41.9)
- added C94: 10n, Capacitor_SMD:C_0603_1608Metric, F.Cu at (20.5, 41.9)
- added C95: 10n, Capacitor_SMD:C_0603_1608Metric, F.Cu at (179.7, 15.3)
- added C96: 10n, Capacitor_SMD:C_0603_1608Metric, F.Cu at (179.7, 17.8)
- added C97: 10n, Capacitor_SMD:C_0603_1608Metric, F.Cu at (179.7, 20.3)
- added C98: 10n, Capacitor_SMD:C_0603_1608Metric, F.Cu at (179.7, 22.8)
- added C99: 20.5nF, Capacitor_SMD:C_0603_1608Metric, F.Cu at (11.3, 44.9)
- added D1: PESD24VL1BLS-QYL, SDM_EV:PESD24VL1BLSQYL-Compact, F.Cu at (25.1, 50.9)
- added D10: BAT54WS-7-F, SDM:SOD2513X120N, F.Cu at (-40.8, 71.4)
- added D11: BAT54WS-7-F, SDM:SOD2513X120N, F.Cu at (-40.8, 74.7)
- added D12: BAT54WS-7-F, SDM:SOD2513X120N, F.Cu at (-40.8, 78.1)
- added D13: PESD24VL1BLS-QYL, SDM_EV:PESD24VL1BLSQYL, F.Cu at (-25.7, 52.8)
- added D14: PESD24VL1BLS-QYL, SDM_EV:PESD24VL1BLSQYL, F.Cu at (-25.7, 56.6)
- added D15: PESD24VL1BLS-QYL, SDM_EV:PESD24VL1BLSQYL, F.Cu at (-21.3, 49.0)
- added D16: PESD24VL1BLS-QYL, SDM_EV:PESD24VL1BLSQYL, F.Cu at (-21.3, 52.8)
- added D17: PESD24VL1BLS-QYL, SDM_EV:PESD24VL1BLSQYL, F.Cu at (-15.7, 42.4)
- added D18: PESD24VL1BLS-QYL, SDM_EV:PESD24VL1BLSQYL, F.Cu at (-11.7, 42.4)
- added D19: PESD24VL1BLS-QYL, SDM_EV:PESD24VL1BLSQYL, F.Cu at (102.6, -7.75)
- added D2: PUSB3FR6Z, SDM:PUSB3FR6Z, F.Cu at (180.4, 66.7)
- added D20: PESD24VL1BLS-QYL, SDM_EV:PESD24VL1BLSQYL, F.Cu at (108.0, -10.2)
- added D21: BAT54WS-7-F, SDM:SOD2513X120N, F.Cu at (150.7, -27.1)
- added D22: BAT54WS-7-F, SDM:SOD2513X120N, F.Cu at (150.7, -24.6)
- added D23: BAT54WS-7-F, SDM:SOD2513X120N, F.Cu at (-35.8, 74.7)
- added D24: BAT54WS-7-F, SDM:SOD2513X120N, F.Cu at (-35.8, 78.1)
- added D25: PESD24VL1BLS-QYL, SDM_EV:PESD24VL1BLSQYL-Compact, F.Cu at (11.3, 50.9)
- added D26: PESD24VL1BLS-QYL, SDM_EV:PESD24VL1BLSQYL-Compact, F.Cu at (14.7, 50.9)
- added D27: BAT54WS-7-F, SDM:SOD2513X120N, F.Cu at (23.5, 47.2)
- added D28: PESD24VL1BLS-QYL, SDM_EV:PESD24VL1BLSQYL-Compact, F.Cu at (18.1, 50.9)
- added D29: PESD24VL1BLS-QYL, SDM_EV:PESD24VL1BLSQYL-Compact, F.Cu at (21.5, 50.9)
- added D3: BAT54WS-7-F, SDM:SOD2513X120N, F.Cu at (27.3, 47.2)
- added D30: PESD24VL1BLS-QYL, SDM_EV:PESD24VL1BLSQYL-Compact, F.Cu at (128.1, 110.1)
- added D31: PESD24VL1BLS-QYL, SDM_EV:PESD24VL1BLSQYL-Compact, F.Cu at (128.1, 113.0)
- added D32: PESD24VL1BLS-QYL, SDM_EV:PESD24VL1BLSQYL-Compact, F.Cu at (128.1, 115.8)
- added D33: PESD24VL1BLS-QYL, SDM_EV:PESD24VL1BLSQYL-Compact, F.Cu at (128.1, 118.7)
- added D4: BAT54WS-7-F, SDM:SOD2513X120N, F.Cu at (31.1, 47.2)
- added D5: BAT54WS-7-F, SDM:SOD2513X120N, F.Cu at (34.9, 47.2)
- added D6: PESD24VL1BLS-QYL, SDM_EV:PESD24VL1BLSQYL-Compact, F.Cu at (28.9, 50.9)
- added D7: PESD24VL1BLS-QYL, SDM_EV:PESD24VL1BLSQYL-Compact, F.Cu at (32.7, 50.9)
- added D8: PESD24VL1BLS-QYL, SDM_EV:PESD24VL1BLSQYL-Compact, F.Cu at (36.5, 50.9)
- added D9: BAT54WS-7-F, SDM:SOD2513X120N, F.Cu at (-45.8, 81.4)
- added FB1: 600Ohm@100MHz ~1.4A, Inductor_SMD:L_0805_2012Metric, F.Cu at (209.3, 69.4)
- added FB2: 600Ohm@100MHz ~1.4A, Inductor_SMD:L_0805_2012Metric, F.Cu at (209.3, 72.1)
- added IC1: MAX20087ATPB_VY+T, SDM_EV:QFN50P400X400X80-21N-D, F.Cu at (210.1, 53.6)
- added IC10: TLP175A_TPL,E, SDM:TLP266J, F.Cu at (139.1, 53.4)
- added IC11: TLP175A_TPL,E, SDM:TLP266J, F.Cu at (4.60, 48.2)
- added IC12: TLP175A_TPL,E, SDM:TLP266J, F.Cu at (124.5, 49.5)
- added IC2: TPS2121RUXR, SDM_Misc:TPS2121RUXR, F.Cu at (198.2, 73.5)
- added IC20: TPD4E05U06QDQARQ1, SDM_EV:DQA_R-PUSON-N10_, F.Cu at (21.2, 16.4)
- added IC24: TPD4E05U06QDQARQ1, SDM_EV:DQA_R-PUSON-N10_, F.Cu at (199.6, 15.3)
- added IC3: TLV76733QWDRBRQ1, SDM_EV:SON65P300X300X100-9N-D, F.Cu at (209.6, 75.9)
- added IC4: MAX20087ATPB_VY+T, SDM_EV:QFN50P400X400X80-21N-D, F.Cu at (210.1, 59.9)
- added IC5: MCP2518FDT-E_SL, SDM_EV:SOIC127P600X175-14N, F.Cu at (94.0, -11.5)
- added IC6: TCAN3413DR, SDM_EV:SOIC127P600X175-8N, F.Cu at (150.9, 44.8)
- added IC7: TLV9064IRUCR, SDM_EV:QFN40P200X200X40-14N, F.Cu at (-6.00, 56.2)
- added IC8: TCAN3413DR, SDM_EV:SOIC127P600X175-8N, F.Cu at (4.40, 42.9)
- added IC9: TCAN3413DR, SDM_EV:SOIC127P600X175-8N, F.Cu at (119.2, 49.7)
- added J3: 6437288-4, SDM_EV:64372884, F.Cu at (11.8, 58.0)
- added J4: 2201778-1, SDM_EV:22017781, F.Cu at (6.62, 17.6)
- added J5: USB4725-03-C-KIT, SDM_Misc:GCT_USB4730-GF-A_REVA, F.Cu at (22.6, 8.60)
- added J6: 6437288-4, SDM_EV:64372884, F.Cu at (54.8, 58.0)
- added L3: 4.7uH, Inductor_SMD:L_SXN_SMDRI62, F.Cu at (191.0, 74.7)
- added LED1: RED, SDM:SSFLXH100LID01, F.Cu at (79.0, 12.8)
- added LED2: GREEN, SDM:SSFLXH100LID01, F.Cu at (72.5, 12.8)
- added LED3: GREEN, SDM:SSFLXH100LID01, F.Cu at (65.8, 12.8)
- added NT1: NetTieGND, NetTie:NetTie-2_SMD_Pad0.5mm, F.Cu at (196.7, 77.2)
- added Q1: DMN62D2UWQ, Package_TO_SOT_SMD:SOT-323_SC-70, F.Cu at (25.0, 44.3)
- added Q2: DMN62D2UWQ, Package_TO_SOT_SMD:SOT-323_SC-70, F.Cu at (28.8, 44.3)
- added Q3: DMN62D2UWQ, Package_TO_SOT_SMD:SOT-323_SC-70, F.Cu at (32.6, 44.3)
- added Q4: DMN62D2UWQ, Package_TO_SOT_SMD:SOT-323_SC-70, F.Cu at (36.4, 44.3)
- added Q5: DMN62D2UWQ, Package_TO_SOT_SMD:SOT-323_SC-70, F.Cu at (-30.3, 73.8)
- added Q6: DMN62D2UWQ, Package_TO_SOT_SMD:SOT-323_SC-70, F.Cu at (-26.3, 60.2)
- added Q7: DMN62D2UWQ, Package_TO_SOT_SMD:SOT-323_SC-70, F.Cu at (-26.3, 63.6)
- added Q8: DMN62D2UWQ, Package_TO_SOT_SMD:SOT-323_SC-70, F.Cu at (-26.3, 67.0)
- added R1: 1k, Resistor_SMD:R_0603_1608Metric, F.Cu at (-15.7, 39.2)
- added R10: 100, Resistor_SMD:R_0603_1608Metric, F.Cu at (35.3, 41.3)
- added R100: 4.75k, Resistor_SMD:R_0603_1608Metric, F.Cu at (16.4, 47.4)
- added R101: 4.75k, Resistor_SMD:R_0603_1608Metric, F.Cu at (19.8, 47.4)
- added R102: 4.75k, Resistor_SMD:R_0603_1608Metric, F.Cu at (191.7, 17.8)
- added R103: 4.75k, Resistor_SMD:R_0603_1608Metric, F.Cu at (191.7, 20.3)
- added R104: 10k, Resistor_SMD:R_0603_1608Metric, F.Cu at (170.8, 65.4)
- added R105: 10k, Resistor_SMD:R_0603_1608Metric, F.Cu at (170.8, 67.9)
- added R106: 100, Resistor_SMD:R_0603_1608Metric, F.Cu at (170.8, 70.4)
- added R107: 100, Resistor_SMD:R_0603_1608Metric, F.Cu at (170.8, 72.9)
- added R108: 100, Resistor_SMD:R_0603_1608Metric, F.Cu at (170.8, 75.4)
- added R11: 5.1k, Resistor_SMD:R_0603_1608Metric, F.Cu at (25.1, 15.6)
- added R12: 100, Resistor_SMD:R_0603_1608Metric, F.Cu at (-46.3, 60.9)
- added R125: 4.75k, Resistor_SMD:R_0603_1608Metric, F.Cu at (191.7, 22.8)
- added R126: 4.75k, Resistor_SMD:R_0603_1608Metric, F.Cu at (191.7, 25.3)
- added R127: 10k, Resistor_SMD:R_0603_1608Metric, F.Cu at (16.4, 50.5)
- added R128: 17.8K, Resistor_SMD:R_0603_1608Metric, F.Cu at (18.1, 47.9)
- added R129: 10k, Resistor_SMD:R_0603_1608Metric, F.Cu at (19.8, 50.5)
- added R13: 100, Resistor_SMD:R_0603_1608Metric, F.Cu at (-46.3, 63.4)
- added R130: 17.8K, Resistor_SMD:R_0603_1608Metric, F.Cu at (21.5, 47.9)
- added R131: 10k, Resistor_SMD:R_0603_1608Metric, F.Cu at (191.7, 37.9)
- added R132: 17.8K, Resistor_SMD:R_0603_1608Metric, F.Cu at (191.7, 40.4)
- added R133: 10k, Resistor_SMD:R_0603_1608Metric, F.Cu at (195.7, 12.8)
- added R134: 17.8K, Resistor_SMD:R_0603_1608Metric, F.Cu at (195.7, 15.3)
- added R135: 10k, Resistor_SMD:R_0603_1608Metric, F.Cu at (195.7, 17.8)
- added R136: 17.8K, Resistor_SMD:R_0603_1608Metric, F.Cu at (195.7, 20.3)
- added R137: 10k, Resistor_SMD:R_0603_1608Metric, F.Cu at (195.7, 22.8)
- added R138: 17.8K, Resistor_SMD:R_0603_1608Metric, F.Cu at (195.7, 25.3)
- added R14: 10k, Resistor_SMD:R_0603_1608Metric, F.Cu at (166.8, 70.4)
- added R15: 100, Resistor_SMD:R_0603_1608Metric, F.Cu at (-46.3, 65.9)
- added R16: 100, Resistor_SMD:R_0603_1608Metric, F.Cu at (153.6, 73.8)
- added R17: 100, Resistor_SMD:R_0603_1608Metric, F.Cu at (2.05, 51.6)
- added R179: 1k, Resistor_SMD:R_0603_1608Metric, F.Cu at (-11.7, 39.2)
- added R18: 100, Resistor_SMD:R_0603_1608Metric, F.Cu at (128.0, 52.1)
- added R181: 1k, Resistor_SMD:R_0603_1608Metric, F.Cu at (100.8, -12.8)
- added R183: 1k, Resistor_SMD:R_0603_1608Metric, F.Cu at (144.0, 39.6)
- added R19: 100, Resistor_SMD:R_0603_1608Metric, F.Cu at (-46.3, 68.4)
- added R2: 0, Resistor_SMD:R_0603_1608Metric, F.Cu at (153.6, 71.3)
- added R20: 100k, Resistor_SMD:R_0603_1608Metric, F.Cu at (26.9, 43.6)
- added R21: 100k, Resistor_SMD:R_0603_1608Metric, F.Cu at (23.1, 43.6)
- added R22: 100k, Resistor_SMD:R_0603_1608Metric, F.Cu at (30.7, 43.6)
- added R23: 100k, Resistor_SMD:R_0603_1608Metric, F.Cu at (34.5, 43.6)
- added R24: 16.2, Resistor_SMD:R_0603_1608Metric, F.Cu at (196.5, 56.7)
- added R25: 5k, Resistor_SMD:R_0603_1608Metric, F.Cu at (196.5, 59.2)
- added R26: 21k, Resistor_SMD:R_0603_1608Metric, F.Cu at (196.5, 61.7)
- added R27: 5k, Resistor_SMD:R_0603_1608Metric, F.Cu at (196.5, 64.2)
- added R28: 100k, Resistor_SMD:R_0603_1608Metric, F.Cu at (-42.3, 58.4)
- added R29: 100k, Resistor_SMD:R_0603_1608Metric, F.Cu at (-42.3, 60.9)
- added R3: 10K, Resistor_SMD:R_0603_1608Metric, F.Cu at (142.3, -30.3)
- added R30: 21k, Resistor_SMD:R_0603_1608Metric, F.Cu at (196.5, 66.7)
- added R31: 5k, Resistor_SMD:R_0603_1608Metric, F.Cu at (196.5, 69.2)
- added R32: 24.2k, Resistor_SMD:R_0603_1608Metric, F.Cu at (200.5, 51.7)
- added R33: 25k, Resistor_SMD:R_0603_1608Metric, F.Cu at (200.5, 54.2)
- added R34: 25k, Resistor_SMD:R_0603_1608Metric, F.Cu at (200.5, 56.7)
- added R35: 100k, Resistor_SMD:R_0603_1608Metric, F.Cu at (-42.3, 63.4)
- added R36: 100k, Resistor_SMD:R_0603_1608Metric, F.Cu at (-42.3, 65.9)
- added R37: 34.8k, Resistor_SMD:R_0603_1608Metric, F.Cu at (200.5, 59.2)
- added R38: 10k, Resistor_SMD:R_0603_1608Metric, F.Cu at (9.60, 50.5)
- added R39: 19.1k, Resistor_SMD:R_0603_1608Metric, F.Cu at (200.5, 61.7)
- added R4: 100, Resistor_SMD:R_0603_1608Metric, F.Cu at (27.7, 41.3)
- added R40: 17.8K, Resistor_SMD:R_0603_1608Metric, F.Cu at (11.3, 47.9)
- added R41: 100k, Resistor_SMD:R_0603_1608Metric, F.Cu at (200.5, 64.2)
- added R42: 1k, Resistor_SMD:R_0603_1608Metric, F.Cu at (200.5, 66.7)
- added R43: 10k, Resistor_SMD:R_0603_1608Metric, F.Cu at (13.0, 50.5)
- added R44: 17.8K, Resistor_SMD:R_0603_1608Metric, F.Cu at (14.7, 47.9)
- added R45: 10K, Resistor_SMD:R_0603_1608Metric, F.Cu at (143.8, -30.3)
- added R46: 1k, Resistor_SMD:R_0603_1608Metric, F.Cu at (27.1, 50.8)
- added R47: 1k, Resistor_SMD:R_0603_1608Metric, F.Cu at (29.2, 47.7)
- added R48: 1k, Resistor_SMD:R_0603_1608Metric, F.Cu at (23.3, 50.8)
- added R49: 1k, Resistor_SMD:R_0603_1608Metric, F.Cu at (25.4, 47.7)
- added R5: 100, Resistor_SMD:R_0603_1608Metric, F.Cu at (23.9, 41.3)
- added R50: 27, Resistor_SMD:R_0603_1608Metric, F.Cu at (25.1, 19.0)
- added R51: 27, Resistor_SMD:R_0603_1608Metric, F.Cu at (25.1, 17.5)
- added R52: 1k, Resistor_SMD:R_0603_1608Metric, F.Cu at (30.9, 50.8)
- added R53: 1k, Resistor_SMD:R_0603_1608Metric, F.Cu at (33.0, 47.7)
- added R54: 1k, Resistor_SMD:R_0603_1608Metric, F.Cu at (34.7, 50.8)
- added R55: 1k, Resistor_SMD:R_0603_1608Metric, F.Cu at (36.8, 47.7)
- added R56: 1k, Resistor_SMD:R_0603_1608Metric, F.Cu at (-38.3, 68.4)
- added R57: 1k, Resistor_SMD:R_0603_1608Metric, F.Cu at (-34.3, 48.4)
- added R58: 1k, Resistor_SMD:R_0603_1608Metric, F.Cu at (-34.3, 50.9)
- added R59: 1k, Resistor_SMD:R_0603_1608Metric, F.Cu at (-34.3, 53.4)
- added R6: 100, Resistor_SMD:R_0603_1608Metric, F.Cu at (31.5, 41.3)
- added R60: 1k, Resistor_SMD:R_0603_1608Metric, F.Cu at (-34.3, 55.9)
- added R61: 1k, Resistor_SMD:R_0603_1608Metric, F.Cu at (-34.3, 58.4)
- added R62: 1k, Resistor_SMD:R_0603_1608Metric, F.Cu at (-34.3, 60.9)
- added R63: 1k, Resistor_SMD:R_0603_1608Metric, F.Cu at (-34.3, 63.4)
- added R64: 10K, Resistor_SMD:R_0603_1608Metric, F.Cu at (146.8, -30.3)
- added R65: 10K, Resistor_SMD:R_0603_1608Metric, F.Cu at (145.3, -30.3)
- added R7: 10k, Resistor_SMD:R_0603_1608Metric, F.Cu at (162.8, 75.4)
- added R79: 5.1k, Resistor_SMD:R_0603_1608Metric, F.Cu at (19.4, 16.4)
- added R8: 10k, Resistor_SMD:R_0603_1608Metric, F.Cu at (162.8, 77.9)
- added R80: 10k, Resistor_SMD:R_0603_1608Metric, F.Cu at (166.8, 75.4)
- added R81: 100, Resistor_SMD:R_0603_1608Metric, F.Cu at (9.60, 39.6)
- added R82: 100, Resistor_SMD:R_0603_1608Metric, F.Cu at (14.5, 39.6)
- added R83: 100, Resistor_SMD:R_0603_1608Metric, F.Cu at (16.4, 39.6)
- added R84: 100, Resistor_SMD:R_0603_1608Metric, F.Cu at (21.3, 39.6)
- added R85: 100, Resistor_SMD:R_0603_1608Metric, F.Cu at (183.7, 37.9)
- added R86: 100, Resistor_SMD:R_0603_1608Metric, F.Cu at (183.7, 40.4)
- added R87: 10k, Resistor_SMD:R_0603_1608Metric, F.Cu at (166.8, 77.9)
- added R88: 100, Resistor_SMD:R_0603_1608Metric, F.Cu at (187.7, 12.8)
- added R89: 100, Resistor_SMD:R_0603_1608Metric, F.Cu at (187.7, 15.3)
- added R9: 10k, Resistor_SMD:R_0603_1608Metric, F.Cu at (166.8, 65.4)
- added R90: 6.49k, Resistor_SMD:R_0603_1608Metric, F.Cu at (9.60, 44.3)
- added R91: 6.49k, Resistor_SMD:R_0603_1608Metric, F.Cu at (13.0, 44.3)
- added R92: 6.49k, Resistor_SMD:R_0603_1608Metric, F.Cu at (16.4, 44.3)
- added R93: 6.49k, Resistor_SMD:R_0603_1608Metric, F.Cu at (19.8, 44.3)
- added R94: 6.49k, Resistor_SMD:R_0603_1608Metric, F.Cu at (187.7, 27.8)
- added R95: 6.49k, Resistor_SMD:R_0603_1608Metric, F.Cu at (187.7, 30.3)
- added R96: 6.49k, Resistor_SMD:R_0603_1608Metric, F.Cu at (187.7, 32.8)
- added R97: 6.49k, Resistor_SMD:R_0603_1608Metric, F.Cu at (187.7, 35.3)
- added R98: 4.75k, Resistor_SMD:R_0603_1608Metric, F.Cu at (9.60, 47.4)
- added R99: 4.75k, Resistor_SMD:R_0603_1608Metric, F.Cu at (13.0, 47.4)
- added RN5: 10k, Resistor_SMD:R_Array_Convex_4x0603, F.Cu at (174.9, 73.6)
- added SW1: SW_Push, Button_Switch_SMD:SW_SPST_CK_KXT3, F.Cu at (175.5, 65.9)
- added SW2: SW_Push, Button_Switch_SMD:SW_SPST_CK_KXT3, F.Cu at (175.5, 69.4)
- added U1: WT0132P4-A1, SDM_EV:WT0132P4-A1, F.Cu at (55.0, 33.9)
- added U17: TLV9064IRUCR, SDM_EV:QFN40P200X200X40-14N, F.Cu at (-10.4, 26.0)
- added U18: TLV9064IRUCR, SDM_EV:QFN40P200X200X40-14N, F.Cu at (-17.9, 105.2)
- added U2: TLV9062xDSG, Package_SON:WSON-8-1EP_2x2mm_P0.5mm_EP0.9x1.6mm_ThermalVias, F.Cu at (12.1, 39.9)
- added U20: LMR51450FSQDRRRQ1, SDM_EV:SON50P300X300X80-13N-D, F.Cu at (209.7, 65.7)
- added U3: TLP293-4, Package_SO:SOIC-16_4.55x10.3mm_P1.27mm, F.Cu at (144.4, -23.3)
- added U4: TLV9062xDSG, Package_SON:WSON-8-1EP_2x2mm_P0.5mm_EP0.9x1.6mm_ThermalVias, F.Cu at (18.9, 39.9)
- added Y1: ECS-3225MVQ-400-BS-TR, SDM_EV:ECS3225MVQ400BSTR, F.Cu at (97.2, -4.95)
Routing:
- net GND: track 0.00 -> 82.2 mm, vias 0 -> 21
- net /A5: track 0.00 -> 32.9 mm
- net /SD1-DAT1: track 0.00 -> 31.8 mm, vias 0 -> 2
- net /SD1-CMD: track 0.00 -> 31.2 mm
- net /A6: track 0.00 -> 30.0 mm
- net /SD1-DAT0: track 0.00 -> 29.8 mm
- net /SD1-CLK: track 0.00 -> 28.7 mm, vias 0 -> 2
- net /A7: track 0.00 -> 28.5 mm
- net /SD1-DAT3: track 0.00 -> 24.3 mm
- net /A8: track 0.00 -> 23.7 mm
- net Net-(D21-K): track 0.00 -> 23.3 mm
- net /SD1-DAT2: track 0.00 -> 22.5 mm
- net Net-(D22-K): track 0.00 -> 21.0 mm
- net /DI3: track 0.00 -> 19.5 mm
- net Net-(U1-USB_DM): track 0.00 -> 17.4 mm
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Other:
- board size 92 x 60 mm -> 87.4 x 70 mm
