File: sdm27ev/sdm27ev-vcu/hardware/sdm27ev-vcu-v1/vcu-can.kicad_sch (KiCad schematic)
At the start: 32 parts, among them IC10 TLP175A_TPL,E, IC11 TCAN3413DR, IC12 TLP175A_TPL,E, IC13 TCAN3413DR, IC14 TLP175A_TPL,E, IC5 MCP2518FDT-E_SL, IC6 TCAN3413DR, IC7 MCP2518FDT-E_SL, IC8 TCAN3413DR, IC9 TLP175A_TPL,E, Y1 ECS-3225MVQ-400-BS-TR, Y2 ECS-3225MVQ-400-BS-TR

Commit message: VCU updates
Updated P4 Symbol
Digital IO protection rework done
Added pending fixes from design review, e.x SDMC pullups
Needs power review - add this to ToDo
Parts:
- removed C26, C27, C28, C29: 100nF, Capacitor_SMD:C_0603_1608Metric, symbol Device:C_Small
- removed IC10: TLP175A_TPL,E, SDM_MiscFootprint:TLP266J, symbol SDM_OPTOCOUPLERS:TLP175A_TPL,E
- removed IC7: MCP2518FDT-E_SL, SOIC127P600X175-14N, symbol SDM_EV:MCP2518FDT-E_SL
- removed IC8: TCAN3413DR, SOIC127P600X175-8N, symbol SDM_EV:TCAN3413DR
- removed R38, R43, R44: 0, Resistor_SMD:R_0402_1005Metric, symbol Device:R_Small
- removed R40: 100, Resistor_SMD:R_0402_1005Metric, symbol Device:R_Small
- removed Y2: ECS-3225MVQ-400-BS-TR, ECS3225MVQ400BSTR, symbol SDM_EV:ECS-3225MVQ-400-BS-TR
Connections:
- net CAN3_STB is gone; now on net GND: IC11.8 (STB)
- net CAN4+ is gone; now on net CAN2+: IC13.7 (CANH), R42.2
- net CAN4- is gone; now on net CAN2-: IC13.6 (CANL), IC14.4
- net CAN4_RX is gone; now on net CAN2_RX: IC13.4 (RXD)
- net CAN4_STB is gone; now on net GND: IC13.8 (STB)
- net CAN4_TERM is gone; now on net CAN2_TERM: IC14.1
- net CAN4_TX is gone; now on net CAN2_TX: IC13.1 (TXD)
- no-connect marks 8 -> 4
Other:
- moved on the sheet: C32, C33, IC13, IC14, R42

Commit message: VCU sch reorg and power rework
Parts:
- renumbered C22 to C1, C23 to C2, C33 to C22, C31 to C23, C24 to C3, C32 to C4, C30 to C5, C25 to C6, IC9 to IC10, IC14 to IC11, IC13 to IC8, IC11 to IC9, R39 to R16, R42 to R17, R41 to R18, R37 to R2
Connections:
- net CAN_SPI2_CS1 renamed CAN_SPI2_CS

Commit message: EV VCU edits, mostly organizational and pre layout/footprint assigned
Parts:
- IC5: footprint SOIC127P600X175-14N -> SDM_EV:SOIC127P600X175-14N
- IC6, IC8, IC9: footprint SOIC127P600X175-8N -> (none)
- R16, R17, R18, R2: footprint Resistor_SMD:R_0402_1005Metric -> Resistor_SMD:R_0603_1608Metric
- Y1: footprint ECS3225MVQ400BSTR -> SDM_EV:ECS3225MVQ400BSTR
