File: sdm27ev/sdm27ev-shutdown-circuit/Shutdown_Circuit/Shutdown_Circuit.kicad_pcb (KiCad board)
At the start: 2 copper layers, 56.9 x 54.6 mm, 18 parts, among them J2 776280-1, K1 PR22-12V-400-1A, K2 PR22-12V-400-1A, K3 PR22-12V-400-1A, Q1 ZXM61N02FTC, Q2 ZXM61N02FTC, Q3 ZXM61N02FTC

Commit message: Added pull down resistors
Parts:
- added R1: 10k, Resistor_SMD:R_0603_1608Metric, F.Cu at (135.7, 79.4)
- added R2: 10k, Resistor_SMD:R_0603_1608Metric, F.Cu at (128.3, 63.5)
- added R3: 10k, Resistor_SMD:R_0603_1608Metric, F.Cu at (129.3, 83.8)
Routing:
- net /BMS KILL SIGNAL: track 5.77 -> 8.98 mm
- net /BSPD KILL SIGNAL: track 20.9 -> 23.8 mm
- net /IMD KILL SIGNAL: track 21.6 -> 23.4 mm
