File: sdm27ev/sdm27ev-shutdown-circuit/Shutdown_Circuit/Shutdown_Circuit.kicad_sch (KiCad schematic)
At the start: 18 parts, among them J2 776280-1, K1 PR22-12V-400-1A, K2 PR22-12V-400-1A, K3 PR22-12V-400-1A, Q1 ZXM61N02FTC, Q2 ZXM61N02FTC, Q3 ZXM61N02FTC

Commit message: Added pull down resistors
Parts:
- added R1, R2, R3: 10k, Resistor_SMD:R_0603_1608Metric, symbol Device:R
Connections:
- net BMS KILL SIGNAL: now also R2.1
- net BSPD KILL SIGNAL: now also R1.1
- net GND: now also R1.2, R2.2, R3.2
- net IMD KILL SIGNAL: now also R3.1
