File: sdm27ev/sdm27ev-vcu/hardware/sdm27ev-vcu-v1/_restore_backup_2026-10-02T21-35-29-444/sdm27ev-vcu-v1.kicad_sch (KiCad schematic)
At the start: 33 parts, among them J1 6437288-1, J2 6437288-1, J4 2201778-1, SW2 SW_Push, SW3 SW_Push, U1 ESP32-P4-Core

Commit message: SDM27 EV VCU Final SCH + docs edit
Parts:
- removed D2: PUSB3FR6Z, PUSB3FR6Z, symbol SDM_MISC:PUSB3FR6Z
- removed LED1: RED, SDM_MiscFootprint:SSFLXH100LID01, symbol SDM_LED:SSF-LXH100LID-01
- removed LED2, LED3: GREEN, SDM_MiscFootprint:SSFLXH100LID01, symbol SDM_LED:SSF-LXH100LID-01
- removed R106, R107, R108: 100, Resistor_SMD:R_0603_1608Metric, symbol Device:R_Small
Connections:
- net StatLED1: no longer names the net of U1.75 (GPIO47)
- net StatLED2: no longer names the net of U1.76 (GPIO48)
- no-connect marks 20 -> 22
Other:
- note removed: "uSD ESD"
- moved on the sheet: C7, C8, J4
