File: sdm27ev/sdm27ev-vcu/hardware/sdm27ev-vcu-v1/_restore_backup_2026-10-02T21-35-29-444/vcu-power.kicad_sch (KiCad schematic)
At the start: 40 parts, among them IC1 TPD4E05U06QDQARQ1, IC2 TPS2121RUXR, IC3 TPS56637RPAR, IC4 TPS61023DRLT, J5 USB4725-03-C-KIT, Q1 RRL035P03FRATR, U3 HUSB238

Commit message: SDM27 EV VCU Final SCH + docs edit
Parts:
- removed R10: 0, Resistor_SMD:R_0603_1608Metric, symbol Device:R_Small
Changed lines of the file:
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@@
 		(color 0 0 0 0)
 	)
-	(junction
-		(at 106.68 33.02)
-		(diameter 0)
-		(color 0 0 0 0)
-	)
 	(no_connect
 		(at 97.79 105.41)
@@
 	(wire
 		(pts
-			(xy 104.14 39.37) (xy 106.68 39.37)
+			(xy 104.14 39.37) (xy 107.95 39.37)
 		)
 		(stroke
@@
 	(wire
 		(pts
-			(xy 97.79 33.02) (xy 95.25 33.02)
-		)
-		(stroke
-			(width 0)
-			(type default)
-		)
-	)
-	(wire
-		(pts
 			(xy 62.23 44.45) (xy 62.23 49.53)
 		)
@@
 	(wire
 		(pts
-			(xy 102.87 33.02) (xy 106.68 33.02)
-		)
-		(stroke
-			(width 0)
-			(type default)
-		)
-	)
-	(wire
-		(pts
 			(xy 119.38 142.24) (xy 119.38 147.32)
 		)
@@
 	(wire
 		(pts
-			(xy 95.25 33.02) (xy 95.25 39.37)
-		)
-		(stroke
-			(width 0)
-			(type default)
-		)
-	)
-	(wire
-		(pts
 			(xy 62.23 102.87) (xy 64.77 102.87)
 		)
@@
 	(wire
 		(pts
-			(xy 106.68 33.02) (xy 106.68 39.37)
-		)
-		(stroke
-			(width 0)
-			(type default)
-		)
-	)
-	(wire
-		(pts
 			(xy 86.36 142.24) (xy 90.17 142.24)
 		)
@@
 	(symbol
 		(lib_id "Device:R_Small")
-		(at 100.33 33.02 90)
-		(mirror x)
-		(unit 1)
-		(body_style 1)
-		(exclude_from_sim no)
-		(in_bom yes)
-		(on_board yes)
-		(in_pos_files yes)
-		(dnp yes)
-		(property "Reference" "R10"
-			(at 100.076 31.496 90)
-			(show_name no)
-			(do_not_autoplace no)
-			(effects
-				(font
-					(size 0.762 0.762)
-				)
-				(justify left)
-			)
-		)
-		(property "Value" "0"
-			(at 101.6 31.496 90)
-			(show_name no)
-			(do_not_autoplace no)
-			(effects
-				(font
-					(size 0.762 0.762)
-				)
-				(justify left)
-			)
-		)
-		(property "Footprint" "Resistor_SMD:R_0603_1608Metric"
-			(at 100.33 33.02 0)
-			(hide yes)
-			(show_name no)
-			(do_not_autoplace no)
-			(effects
-				(font
-					(size 1.27 1.27)
-				)
-			)
-		)
-		(property "Datasheet" ""
-			(at 100.33 33.02 0)
-			(hide yes)
-			(show_name no)
-			(do_not_autoplace no)
-			(effects
-				(font
-					(size 1.27 1.27)
-				)
-			)
-		)
-		(property "Description" "Resistor, small symbol"
-			(at 100.33 33.02 0)
-			(hide yes)
-			(show_name no)
-			(do_not_autoplace no)
-			(effects
-				(font
-					(size 1.27 1.27)
-				)
-			)
-		)
-		(pin "2"
-		)
-		(pin "1"
-		)
-		(instances
-			(project "sdm27ev-vcu-v1"
-				(path "/aaff56d4-6a2c-4b9b-8d6c-def2b75cacc9/6a2ee1fd-03b1-4da7-bb6a-9a75b73da95c"
-					(reference "R10")
-					(unit 1)
-				)
-			)
-		)
-	)
-	(symbol
-		(lib_id "Device:R_Small")
 		(at 95.25 41.91 0)
 		(mirror x)
@@
 			)
 		)
-		(property "Datasheet" "https://www.hynetek.com/uploadfiles/site/219/news/aabbbbdb-48c9-4a44-a6dc-2c15f53282e6.pdf"
+		(property "Datasheet" ""
 			(at 74.93 41.91 0)
 			(hide yes)
@@
 	(symbol
 		(lib_id "power:VBUS")
-		(at 106.68 33.02 0)
+		(at 107.95 39.37 0)
 		(unit 1)
 		(body_style 1)
@@
 		(dnp no)
 		(property "Reference" "#PWR04"
-			(at 106.68 36.83 0)
+			(at 107.95 43.18 0)
 			(hide yes)
 			(show_name no)
@@
 		)
 		(property "Value" "VBUS"
-			(at 106.68 29.464 0)
+			(at 107.95 35.814 0)
 			(show_name no)
 			(do_not_autoplace no)
@@
 		)
 		(property "Footprint" ""
-			(at 106.68 33.02 0)
+			(at 107.95 39.37 0)
 			(hide yes)
 			(show_name no)
@@
 		)
 		(property "Datasheet" ""
-			(at 106.68 33.02 0)
+			(at 107.95 39.37 0)
 			(hide yes)
 			(show_name no)
@@
 		)
 		(property "Description" "Power symbol creates a global label with name \"VBUS\""
-			(at 106.68 33.02 0)
+			(at 107.95 39.37 0)
 			(hide yes)
 			(show_name no)
