File: sdm27ev/smd27ev-discharge-circuit/Discharge Circuit.kicad_sch (KiCad schematic)
At the start: 7 parts, among them J1 MPT-02-01-XX-X-RA-SD, J2 IPBT-102-H1-T-S-RA-K, J3 PET-02-01-T-VT-LC, K2 FTR-E1AA012Y-GR

Commit message: Fixed discharge relay symbol/footprint
Parts:
- removed K2: FTR-E1AA012Y-GR, FTR-E1AA012Y-GR:FTRE1AA012YGR, symbol FTR-E1AA012Y-GR:FTR-E1AA012Y-GR
- added K1: (no value), footprint:S82405VHR, symbol S8-121B04:S8-121B04
Connections:
- net GND: now also K1.2 (-)
- net at J1.1: now also K1.3 (NC)
- net at J3.2: now also K1.4 (NC)
- net at D1.1 (K), J2.1: now also K1.1 (+)
