File: sdm27ev/sdm27ev-esf-tracive-system-schematics/Shutdown_Circuit_Full_ESF.kicad_sch (KiCad schematic)
At the start: 44 parts, among them J1 Precharge/Relay_Controller, K1 PR22-12V-400-1A, K2 PR22-12V-400-1A, K3 PR22-12V-400-1A, K4 Main Contactor Relay, K5 Isolation_Relay_+, K6 Isolation Relay -, K7 Precharge Relay, K8 Discharge Relay, Q1 ZXM61N02FTC, Q2 ZXM61N02FTC, Q3 ZXM61N02FTC, SW1 GLVMS, SW2 Inertia_Switch, SW3 Cockpit_Shutdown_Button, SW4 Right_Shutdown_Button, SW5 Left_Shutdown_Button, SW6 BOTS, SW7 TSMS, SW8 TS_Container_Interlock

Commit message: move glv 12V after fuse
Connections:
- net +12V: now also D1.1 (K), D2.1 (K), D3.1 (K), K1.1 (COIL_1), K1.2 (COM_1), K2.1 (COIL_1), K3.1 (COIL_1), SW1.2 (B); no longer F1.1, GLV_Battery.1 (+)
- new net: F1.1, GLV_Battery.1 (+)
