File: sdm27ev/sdm27ev-esf-tracive-system-schematics/Charging TS Schematic.kicad_sch (KiCad schematic)
At the start: 21 parts, among them K1 AIR +, K2 AIR -

Commit message: Added/FIxed ESF connectors Tractive system & Charger
Parts:
- added F11: Schurter 8020.5070.G 5A, symbol Device:Fuse
Other:
- note added: "HVSL1000022A1HB"
- note added: "McMaster-Carr 5340N21"
- note removed: "NEED TO FIX"
Changed lines of the file:
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@@
-	)
-	(rectangle
-		(start 172.72 45.72)
-		(end 193.04 50.8)
-		(stroke
-			(width 0)
-			(type solid)
-			(color 0 0 0 1)
-		)
-		(fill
-			(type none)
-		)
 	)
 	(rectangle
@@
 	)
 	(rectangle
-		(start 266.7 68.58)
+		(start 246.38 68.58)
 		(end 276.86 76.2)
 		(stroke
@@
 		(start 215.9 68.58)
 		(end 223.774 76.2)
-		(stroke
-			(width 0)
-			(type solid)
-			(color 0 0 0 1)
-		)
-		(fill
-			(type none)
-		)
-	)
-	(rectangle
-		(start 246.38 71.12)
-		(end 254.254 78.74)
 		(stroke
 			(width 0)
@@
 		)
 	)
-	(text "NEED TO FIX"
-		(exclude_from_sim no)
-		(at 50.038 37.084 0)
-		(effects
-			(font
-				(size 2.54 2.54)
-				(thickness 0.508)
-				(bold yes)
-			)
-		)
-	)
 	(text "12V\n"
 		(exclude_from_sim no)
@@
 			(font
 				(size 2.032 2.032)
+			)
+		)
+	)
+	(text "McMaster-Carr\n5340N21"
+		(exclude_from_sim no)
+		(at 261.366 66.294 0)
+		(effects
+			(font
+				(size 1.27 1.27)
 			)
 		)
@@
 		)
 	)
+	(text "HVSL1000022A1HB"
+		(exclude_from_sim no)
+		(at 232.156 67.056 0)
+		(effects
+			(font
+				(size 1.27 1.27)
+			)
+		)
+	)
 	(junction
 		(at 87.63 50.8)
@@
 	(wire
 		(pts
-			(xy 193.04 88.9) (xy 193.04 92.71)
+			(xy 193.04 88.9) (xy 193.04 93.98)
 		)
 		(stroke
@@
 			(width 0.508)
 			(type default)
-		)
-	)
-	(wire
-		(pts
-			(xy 193.04 49.53) (xy 231.14 49.53)
-		)
-		(stroke
-			(width 0)
-			(type default)
-			(color 21 205 210 1)
 		)
 	)
@@
 			(width 0.381)
 			(type solid)
+		)
+	)
+	(wire
+		(pts
+			(xy 175.26 50.8) (xy 248.92 50.8)
+		)
+		(stroke
+			(width 0)
+			(type default)
+			(color 21 205 210 1)
 		)
 	)
@@
 	(wire
 		(pts
-			(xy 231.14 92.71) (xy 231.14 49.53)
+			(xy 248.92 93.98) (xy 248.92 50.8)
 		)
 		(stroke
@@
 	(wire
 		(pts
-			(xy 193.04 92.71) (xy 231.14 92.71)
+			(xy 193.04 93.98) (xy 248.92 93.98)
 		)
 		(stroke
@@
 			(type default)
 			(color 255 155 3 1)
+		)
+	)
+	(wire
+		(pts
+			(xy 175.26 45.72) (xy 175.26 50.8)
+		)
+		(stroke
+			(width 0)
+			(type default)
+			(color 21 205 210 1)
 		)
 	)
@@
 					(unit 1)
 				)
+			)
+		)
+	)
+	(symbol
+		(lib_id "Device:Fuse")
+		(at 185.42 38.1 90)
+		(unit 1)
+		(body_style 1)
+		(exclude_from_sim no)
+		(in_bom yes)
+		(on_board yes)
+		(in_pos_files yes)
+		(dnp no)
+		(property "Reference" "F11"
+			(at 185.42 42.164 90)
+			(show_name no)
+			(do_not_autoplace no)
+			(effects
+				(font
+					(size 1.27 1.27)
+				)
+			)
+		)
+		(property "Value" "Schurter 8020.5070.G 5A"
+			(at 187.96 40.132 90)
+			(show_name no)
+			(do_not_autoplace no)
+			(effects
+				(font
+					(size 1.27 1.27)
+				)
+			)
+		)
+		(property "Footprint" ""
+			(at 185.42 39.878 90)
+			(hide yes)
+			(show_name no)
+			(do_not_autoplace no)
+			(effects
+				(font
+					(size 1.27 1.27)
+				)
+			)
+		)
+		(property "Datasheet" ""
+			(at 185.42 38.1 0)
+			(hide yes)
+			(show_name no)
+			(do_not_autoplace no)
+			(effects
+				(font
+					(size 1.27 1.27)
+				)
+			)
+		)
+		(property "Description" "Fuse"
+			(at 185.42 38.1 0)
+			(hide yes)
+			(show_name no)
+			(do_not_autoplace no)
+			(effects
+				(font
+					(size 1.27 1.27)
+				)
+			)
+		)
+		(pin "2"
+		)
+		(pin "1"
+		)
+		(instances
+			(project "TS System Schematic"
+				(path "/b2aeb17e-134d-4155-8140-6b03f1864ab3/8949d33a-b98a-43ca-b87d-179eb107db00"
+					(reference "F11")
+					(unit 1)
+				)
