File: sdm27ev/sdm27ev-esf-tracive-system-schematics/TS System Schematic.kicad_sch (KiCad schematic)
At the start: 2 parts

Commit message: Added/FIxed ESF connectors Tractive system & Charger
Other:
- note added: "HVSL1000022A1HB"
- note added: "McMaster-Carr 5340N21"
Changed lines of the file:
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@@
+		)
+	)
+	(text "McMaster-Carr\n5340N21"
+		(exclude_from_sim no)
+		(at 46.228 93.472 0)
+		(effects
+			(font
+				(size 1.27 1.27)
+			)
 		)
 	)
@@
 			(font
 				(size 2.54 2.54)
+			)
+		)
+	)
+	(text "McMaster-Carr\n5340N21"
+		(exclude_from_sim no)
+		(at 68.834 100.838 0)
+		(effects
+			(font
+				(size 1.27 1.27)
+			)
+		)
+	)
+	(text "McMaster-Carr\n5340N21"
+		(exclude_from_sim no)
+		(at 106.426 105.156 0)
+		(effects
+			(font
+				(size 1.27 1.27)
 			)
 		)
@@
 			)
 		)
+	)
+	(text "HVSL1000022A1HB"
+		(exclude_from_sim no)
+		(at 65.278 28.448 0)
+		(effects
+			(font
+				(size 1.27 1.27)
+			)
+		)
