File: sdm27ev/sdm27ev-tssi/TSSI_v2.1.kicad_pcb (KiCad board)
At the start: 2 copper layers, 75.7 x 53.7 mm, 49 parts, among them IC1 MIC37100-3.3WS, IC2 ESP32-S3-WROOM-1-N8R8, J1 776267-1, J3 USB_B_Micro, J4 SSQ-103-03-G-D, Q1 LTV-817S-TA1, Q2 LTV-817S-TA1, Q3 LTV-817S-TA1, U1 LM2575HVS-5.0_NOPB, U3 USBLC6-2SC6, U4 TPS3702, U5 AO3400A, U6 AO3400A

Commit message: Added TSSI Testpoints
Parts:
- added BLACK_TP1: 5006, SDM Footprints:5006, F.Cu at (190.8, 85.1)
- added RED_TP1: 5005, SDM Footprints:5005, F.Cu at (190.9, 91.5)
- added WHITE_TP1: 5007, SDM Footprints:5007, F.Cu at (128.4, 110.9)
- added WHITE_TP2: 5007, SDM Footprints:5007, F.Cu at (128.3, 121.0)
- added WHITE_TP3: 5007, SDM Footprints:5007, F.Cu at (128.3, 116.0)
- added WHITE_TP4: 5007, SDM Footprints:5007, F.Cu at (192.0, 118.1)
- renumbered J4 to J2
Routing:
- net /BMS_CHECK: track 36.0 -> 69.3 mm
- net +3.3V: track 131.0 -> 150.5 mm, vias 4 -> 6
- net /IMD_CHECK: track 47.0 -> 61.3 mm, vias 2 -> 4
- net /ENABLE: track 35.1 -> 42.3 mm
- net /LAMP_CHECK: track 60.7 -> 66.4 mm
- net /GPIO39: track 54.9 -> 55.6 mm
- net GND: vias 54 -> 55
