File: sdm27ev/sdm27ev-tssi/TSSI_v2.1.kicad_sch (KiCad schematic)
At the start: 49 parts, among them IC1 MIC37100-3.3WS, IC2 ESP32-S3-WROOM-1-N8R8, J1 776267-1, J3 USB_B_Micro, J4 SSQ-103-03-G-D, Q1 LTV-817S-TA1, Q2 LTV-817S-TA1, Q3 LTV-817S-TA1, U1 LM2575HVS-5.0_NOPB, U3 USBLC6-2SC6, U4 TPS3702, U5 AO3400A, U6 AO3400A

Commit message: Added TSSI Testpoints
Parts:
- added BLACK_TP1: 5006, SDM Footprints:5006, symbol SDM Symbols:5006
- added RED_TP1: 5005, SDM Footprints:5005, symbol SDM Symbols:5005
- added WHITE_TP1, WHITE_TP2, WHITE_TP3, WHITE_TP4: 5007, SDM Footprints:5007, symbol SDM Symbols:5007
- renumbered J4 to J2
Connections:
- net +3.3V: now also RED_TP1.1
- net BMS_CHECK: now also WHITE_TP1.1
- net ENABLE: now also WHITE_TP4.1
- net GND: now also BLACK_TP1.1
- net IMD_CHECK: now also WHITE_TP2.1
- net LAMP_CHECK: now also WHITE_TP3.1
