File: sdm27ev/sdm27ev-accumulator-pack/SDM_AccumulatorPack.kicad_sch (KiCad schematic)
At the start: 16 parts, among them K6 AIR -, K7 Discharge Relay, K8 AIR +, K9 Precharge Relay, U5 Precharge Control, U6 Energy Meter, U7 IMD, U8 Voltage Indicator

Commit message: Add files via upload
Finished Switching the AIRS and most of the stuff
Connections:
- net at U6. (Interlock_B): now also R7.1, TP3.1
Other:
- added sheet Version 1.2 (Version 1.2.kicad_sch)
Changed lines of the file:
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@@
+		)
+	)
+	(sheet
+		(at 374.65 274.32)
+		(size 384.81 218.44)
+		(exclude_from_sim no)
+		(in_bom yes)
+		(on_board yes)
+		(dnp no)
+		(fields_autoplaced yes)
+		(stroke
+			(width 0.1524)
+			(type solid)
+		)
+		(fill
+			(color 0 0 0 0)
+		)
+		(property "Sheetname" "Version 1.2"
+			(at 374.65 273.6084 0)
+			(show_name no)
+			(do_not_autoplace no)
+			(effects
+				(font
+					(size 1.27 1.27)
+				)
+				(justify left bottom)
+			)
+		)
+		(property "Sheetfile" "Version 1.2.kicad_sch"
+			(at 374.65 493.3446 0)
+			(show_name no)
+			(do_not_autoplace no)
+			(effects
+				(font
+					(size 1.27 1.27)
+				)
+				(justify left top)
+			)
+		)
+		(instances
+			(project "SDM_AccumulatorPack"
+				(path "/b2e70c53-29d1-4b3b-8053-28286598a524"
+					(page "3")
+				)
+			)
 		)
 	)
