File: sdm27ev/sdm27ev-accumulator-pack/untitled.kicad_sch (KiCad schematic)
At the start: 38 parts, among them J1 Conn_01x04_Pin, K1 Discharge Relay, K2 AIR -, K4 AIR +, K5 Precharge Relay, SW1 SW_SPST, SW2 SW_SPST, SW3 SW_SPST, SW4 SW_SPST, SW5 SW_SPST, SW6 SW_SPST, SW7 SW_SPST, SW8 SW_SPST, U1 IMD, U17 Energy Meter, U18 Temp_BT6, U19 Temp_BT7, U2 Voltage Indicator, U20 Temp_BT8, U21 Temp_BT9, U22 Temp_BT10, U23 Temp_BT11, U3 Temp_BT2, U4 Precharge Control

Commit message: Add files via upload
Finished Switching the AIRS and most of the stuff
Parts:
- added R4: Discharge Resistor, symbol Device:R
- U18: value Temp_BT6 -> Temp_BT10
- U19: value Temp_BT7 -> Temp_BT9
- U21: value Temp_BT9 -> Temp_BT7
- U22: value Temp_BT10 -> Temp_BT6
- U23: value Temp_BT11 -> Temp_BT2
- U3: value Temp_BT2 -> Temp_BT11
Connections:
- net TSMP+ is gone; now on net TSMP +: J1.TS+
- net TSMP- is gone; now on net TSMP -: J1.TS-
- net BAT -: now also R3.2; no longer K1.4
- net TSMP +: now also K1.1; no longer K5.1
- net TSMP -: now also K5.1, R4.2
- net at U4.2 (OUT): now also K2.2; no longer K4.2
- net at F2.2, K4.1: no longer R3.2
- net at F2.1, SW8.1 (A): no longer K1.1
- net CTRL_IN renamed SDC_AIR
- net SDC_AIR: now also K4.2; no longer K2.2
- new net: K1.4, R4.1
Other:
- moved on the sheet: BT10, BT11, BT2, BT6, BT7, BT8, BT9, Current_Sensor, F2, J1, K1, K2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
