File: sdm27ev/sdm27ev-bspd-v1.2/BSPD_V1.2_EV.kicad_sch (KiCad schematic)
At the start: 53 parts, among them IC2 LM2901BIRTER, IC3 74AHC1G08, IC4 SN74HC32PWR, IC5 L7805ACD2T-TR, IC6 SN74LVC1G17DBVRG4, J1 776280-1, Q1 2N7002,215

Commit message: move glv 12V after fuse
Parts:
- BLACK_TP1: symbol SDM_TESTPOINT:5006 -> SDM_MiscSymbol:5006
- D2, D3, D4, D5, D6: symbol SDM_DIODES:BAT54XV2T1G -> SDM_MiscSymbol:BAT54XV2T1G
- D7: symbol SDM_SCR:X0202MN_5BA4 -> SDM_MiscSymbol:X0202MN_5BA4
- IC2: symbol SDM_COMPARITOR:LM2901BIRTER -> SDM_MiscSymbol:LM2901BIRTER
- IC3: symbol SDM_LOGIC:74AHC1G08GW,125 -> SDM_MiscSymbol:74AHC1G08GW,125
- IC4: symbol SDM_LOGIC:SN74HC32PWR -> SDM_MiscSymbol:SN74HC32PWR
- IC5: symbol SDM_VOLTAGE_REGULATORS:L7805ACD2T-TR -> SDM_MiscSymbol:L7805ACD2T-TR
- IC6: footprint Misc:SOT95P280X145-5N -> SOT95P280X145-5N
- J1: symbol SDM_CONNECTOR:776280-1 -> SDM_MiscSymbol:776280-1
- LED1, LED2: symbol SDM_LED:150060RS75000 -> SDM_MiscSymbol:150060RS75000
- LED4, LED5, LED6, LED7, LED8, LED9: symbol SDM_LED:150060GS75000 -> SDM_MiscSymbol:150060GS75000
- Q1: symbol SDM_MOSFET_N-CHANNEL:2N7002,215 -> SDM_MiscSymbol:2N7002,215
- RED_TP3, RED_TP4, RED_TP5, RED_TP6: symbol SDM_TESTPOINT:5005 -> SDM_MiscSymbol:5005
- VR3, VR4, VR5, VR6: symbol SDM_VARIABLE_RESISTOR:3386P-1-103TLF -> SDM_MiscSymbol:3386P-1-103TLF
- WHITE_TP1, WHITE_TP2: symbol SDM_TESTPOINT:5007 -> SDM_MiscSymbol:5007
Connections:
- no-connect marks 6 -> 4

Commit message: Tentitive Schematic for BSPD
Changed lines of the file:
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@@
 		)
 		(property "Value" "GND"
-			(at 148.59 34.29 0)
+			(at 135.89 48.26 0)
 			(show_name no)
 			(do_not_autoplace no)
