File: sdm27ev/sdm27ev-bspd-v2/Current Sensor.kicad_sch (KiCad schematic)
At the start: 21 parts, among them U1 TLV9022QDRQ1, U2 LTV-827S

Commit message: Tentitive Schematic for BSPD
Parts:
- added R201: 10K, symbol Device:R
- renumbered C1 to C201, C2 to C202, H1 to H201, H2 to H202, H3 to H203, H4 to H204, LED7 to LED201, LED6 to LED202, R1 to R202, R2 to R203, R3 to R204, R4 to R205, R6 to R206, R5 to R207, RED_TP1 to RED_TP201, RED_TP2 to RED_TP202, U1 to U201, U2 to U202, VR1 to VR201, VR2 to VR202, WHITE_TP1 to WHITE_TP201
Connections:
- net CH1_CURRENT SENSOR: now also R201.2
- net GND_BMS: now also R201.1
- net POWER UNDER FAUT renamed Current Sensor Fault
- net ~{Under Current Fault} renamed ~{Current Sensor Fault}

Commit message: Reflow numbers and page order
Parts:
- renumbered C201 to C301, C202 to C302, H201 to H301, H202 to H302, H203 to H303, H204 to H304, LED201 to LED301, LED202 to LED302, R201 to R301, R202 to R302, R203 to R303, R204 to R304, R205 to R305, R206 to R306, R207 to R307, RED_TP201 to RED_TP301, RED_TP202 to RED_TP302, U201 to U301, U202 to U302, VR201 to VR301, VR202 to VR302, WHITE_TP201 to WHITE_TP301

Commit message: small referance changes
Parts:
- C301, C302: footprint (none) -> Capacitor_SMD:C_0603_1608Metric
- H301, H302, H303, H304: footprint (none) -> MountingHole:MountingHole_2.2mm_M2_DIN965_Pad
- R301, R302, R303, R304, R305, R306, R307: footprint (none) -> Resistor_SMD:R_0603_1608Metric
- WHITE_TP301: Measure HES -> Current Sensor
Connections:
- net +5V: now also U302.6, U302.8; no longer U302.6, U302.8
- net Current Sensor Fault: now also U302.7; no longer U302.5
- net POWER OVER FAUT: now also U302.5; no longer U302.7
- net ~{Current Sensor Fault}: now also U302.2; no longer U302.4
- net ~{Over Current Fault}: now also U302.4; no longer U302.2
- net at R303.1: now also U302.1; no longer U302.3
- net at R302.2: now also U302.3; no longer U302.1
Changed lines of the file:
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@@
 			)
 		)
-		(property "Footprint" ""
+		(property "Footprint" "Resistor_SMD:R_0603_1608Metric"
 			(at 50.8 145.288 90)
 			(hide yes)
@@
 			)
 		)
-		(property "Footprint" ""
+		(property "Footprint" "MountingHole:MountingHole_2.2mm_M2_DIN965_Pad"
 			(at 142.24 193.04 0)
 			(hide yes)
@@
 			)
 		)
-		(property "Footprint" ""
+		(property "Footprint" "MountingHole:MountingHole_2.2mm_M2_DIN965_Pad"
 			(at 142.24 173.99 0)
 			(hide yes)
@@
 			)
 		)
-		(property "Footprint" ""
+		(property "Footprint" "Resistor_SMD:R_0603_1608Metric"
 			(at 39.37 145.288 90)
 			(hide yes)
@@
 			)
 		)
-		(property "Footprint" ""
+		(property "Footprint" "Resistor_SMD:R_0603_1608Metric"
 			(at 57.15 122.428 90)
 			(hide yes)
@@
 			)
 		)
-		(property "Footprint" ""
+		(property "Footprint" "Resistor_SMD:R_0603_1608Metric"
 			(at 31.75 122.428 90)
 			(hide yes)
@@
 			)
 		)
-		(property "Footprint" ""
+		(property "Footprint" "Resistor_SMD:R_0603_1608Metric"
 			(at 63.5 163.068 90)
 			(hide yes)
@@
 			)
 		)
-		(property "Footprint" ""
+		(property "Footprint" "Capacitor_SMD:C_0603_1608Metric"
 			(at 20.32 94.2848 0)
 			(hide yes)
@@
 			)
 		)
-		(property "Footprint" ""
+		(property "Footprint" "MountingHole:MountingHole_2.2mm_M2_DIN965_Pad"
 			(at 142.24 180.34 0)
 			(hide yes)
@@
 		(lib_id "Isolator:LTV-827S")
 		(at 49.53 128.27 270)
-		(unit 2)
+		(unit 1)
 		(body_style 1)
 		(exclude_from_sim no)
@@
 				(path "/f5fc7189-56d7-49a3-a293-889ea2ed3485/e2198b7f-9f60-4a5d-be1e-3151c1f6d596"
 					(reference "U302")
-					(unit 2)
+					(unit 1)
 				)
 			)
@@
 			)
 		)
-		(property "Measure" "HES"
+		(property "Measure" "Current Sensor"
 			(at 103.124 39.878 0)
 			(hide yes)
@@
 			)
 		)
-		(property "Footprint" ""
+		(property "Footprint" "Resistor_SMD:R_0603_1608Metric"
 			(at 91.948 49.53 90)
 			(hide yes)
@@
 		(at 40.64 128.27 90)
 		(mirror x)
-		(unit 1)
+		(unit 2)
 		(body_style 1)
 		(exclude_from_sim no)
@@
 		(dnp no)
 		(property "Reference" "U302"
-			(at 32.512 127.254 90)
+			(at 29.718 127 90)
 			(show_name no)
 			(do_not_autoplace no)
@@
 				(path "/f5fc7189-56d7-49a3-a293-889ea2ed3485/e2198b7f-9f60-4a5d-be1e-3151c1f6d596"
 					(reference "U302")
-					(unit 1)
+					(unit 2)
 				)
 			)
@@
 			)
 		)
-		(property "Footprint" ""
+		(property "Footprint" "Capacitor_SMD:C_0603_1608Metric"
 			(at 20.32 81.5848 0)
 			(hide yes)
@@
 			)
 		)
-		(property "Footprint" ""
+		(property "Footprint" "MountingHole:MountingHole_2.2mm_M2_DIN965_Pad"
 			(at 142.24 186.69 0)
 			(hide yes)
@@
 			)
 		)
-		(property "Footprint" ""
+		(property "Footprint" "Resistor_SMD:R_0603_1608Metric"
 			(at 26.67 163.068 90)
 			(hide yes)

Commit message: Updated BSPD Schematic
Other:
- note added: "Brightness: 10mcd ΔV = 5V - 2.7V = 2.3V V/I = 2.3V / 0.5mA = 4.6kΩ ≈ 4.7kΩ LED Current Draw: 0.5mA"
- note removed: "Brightness: 10mcd ΔV = 5V - 2.7V = 2.3V V/I = 2.3V / 0.5mA = 4600Ω 4.6k ≈ 4.7kΩ LED Current Draw: 0.5mA"
Changed lines of the file:
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@@
 		)
 	)
-	(text "Brightness: 10mcd\nΔV = 5V - 2.7V = 2.3V\nV/I = 2.3V / 0.5mA = 4600Ω\n4.6k ≈ 4.7kΩ\nLED Current Draw: 0.5mA"
+	(text "Brightness: 10mcd\nΔV = 5V - 2.7V = 2.3V\nV/I = 2.3V / 0.5mA =\n  4.6kΩ ≈ 4.7kΩ\nLED Current Draw: 0.5mA"
 		(exclude_from_sim no)
 		(at 17.526 173.736 0)
