File: sdm27ev/sdm27ev-bspd-v2/sdm27ev-bspd-v2.kicad_pcb (KiCad board)
At the start: 2 copper layers, 40 x 40 mm, 66 parts, among them IC201 74AHC1G08, IC202 SN74LVC1G17DBVRG4, IC203 SN74HC32PWR, IC204 L7805ACD2T-TR, J101 776280-1, J102 776280-1, U201 TLV9022QDRQ1, U301 TLV9022QDRQ1, U302 LTV-827S

Commit message: routing lights cleaner
Parts:
- moved R306 21.1 mm to (56.0, 148.2), turned to -90 degrees
- moved R305 17.1 mm to (53.8, 131.0)
- moved LED301 16.8 mm to (55.0, 146.0), turned to 180 degrees
- moved R304 7.40 mm to (54.8, 144.0)
- moved LED302 3.21 mm to (49.2, 147.5)
- moved R307 3.00 mm to (45.8, 147.7)
- moved R302 2.50 mm to (44.5, 128.0)
- moved R303 2.50 mm to (44.5, 131.0)
- moved U302 2.50 mm to (49.8, 137.5)
- moved Dylan Shah 1.10 mm to (54.1, 128.3)
Routing:
- net /Current Sensor Fault: track 24.8 -> 32.7 mm
- net /POWER OVER FAUT: track 32.0 -> 27.8 mm
- net +5V_BMS: track 72.6 -> 76.2 mm
- net +5V: track 41.1 -> 44.5 mm
- net /Current Sensor Sub-Board/~{Over Current Fault}: track 13.5 -> 11.1 mm
- net /Current Sensor Sub-Board/~{Current Sensor Fault}: track 12.0 -> 9.66 mm
- net GND: track 6.28 -> 4.75 mm, vias 49 -> 58
- net Net-(LED302-K): track 1.60 -> 2.37 mm
- net GND_BMS: vias 90 -> 79
Other:
- board text removed: "BSPD SIDE"

Commit message: Updated BSPD Schematic
Parts:
- added G***: LOGO, SDM_MiscFootprint:SDM EV LOGO, B.Cu at (30.8, 135.8)
- added G***: LOGO, SDM_MiscFootprint:Robocat 10x10mm, B.Cu at (24.2, 148.0)
Other:
- board text added: "Falstad Simulation:"
- board text added: "Pinout: 1 - >5kW Fault 2 - Sensor DC 3 - BSPD GND 4 - BSPD 5V 5 - NC 6 - BMS 5V 7 - Current Sensor Ch1 8 - BMS GND"
- board text added: "SDM EV '27 BSPD V2 Dylan Shah Carter Kortan"
