File: sdm27ev/sdm27ev-precharge/prechargecontrol/prechargecontrol.kicad_sch (KiCad schematic)
At the start: 0 parts

Commit message: Precharge control pcb schem v1
Parts:
- added C1, C5, C6: 22uF, symbol Device:C
- added C10, C11, C14, C16: 10uF, symbol Device:C
- added C12, C13, C15, C17, C19, C20, C22, C23, C25, C30, C4, C9: 100nF, symbol Device:C
- added C18, C21: 100pF, symbol Device:C
- added C2: 2.2uF, symbol Device:C
- added C24: 4.7uF, symbol Device:C
- added C26, C27, C28, C29, C3, C31, C7, C8: 1uF, symbol Device:C
- added D1: SS1H10-E3/61T, symbol Device:D
- added D2: SMBJ18A, symbol Device:D_Zener
- added D3: SMAJ40CA-E3/5A, symbol Device:D_TVS
- added D4, D5: SS14 / DNP, symbol Device:D
- added D6: GREEN, symbol Device:LED
- added D7: YELLOW, symbol Device:LED
- added D8: RED, symbol Device:LED
- added D9: GREEN / 3V3, symbol Device:LED
- added F1: FUSE_TBD, symbol Device:Fuse
- added J1: GLV_INPUT, symbol Connector_Generic:Conn_01x02
- added J2: PACK_VSENSE, symbol Connector_Generic:Conn_01x02
- added J3: DC_LINK_VSENSE, symbol Connector_Generic:Conn_01x02
- added J4: PRECHARGE_RELAY, symbol Connector_Generic:Conn_01x02
- added J5: SWD, symbol Connector_Generic:Conn_01x05
- added J6: MAIN_AIR, symbol Connector_Generic:Conn_01x02
- added J7: RESERVED / DNP, symbol Connector_Generic:Conn_01x02
- added J8: SDC_COIL_POWER, symbol Connector_Generic:Conn_01x02
- added L1: 22uH, symbol Device:L
- added Q1: IRL640PBF, symbol Transistor_FET:Q_NMOS_GDS
- added Q2: IRL540NPBF, symbol Transistor_FET:Q_NMOS_GDS
- added Q3: AO3400A / DNP, symbol Transistor_FET:Q_NMOS_GSD
- added R1: 0R, symbol Device:R
- added R10, R11, R12, R13: 1k, symbol Device:R
- added R14, R15, R16, R17, R4, R5: 10k, symbol Device:R
- added R2: 100k, symbol Device:R
- added R3: 24.9k, symbol Device:R
- added R6: 10k / DNP, symbol Device:R
- added R7, R8: 100, symbol Device:R
- added R9: 100 / DNP, symbol Device:R
- added TP1: SDC_COIL, symbol Connector:TestPoint
- added TP2, TP4: (no value), symbol Connector:TestPoint
- added TP3, TP5, TP6: TestPoint, symbol Connector:TestPoint
- added TP7: PRECHARGE_CMD, symbol Connector:TestPoint
- added TP8: MAIN_CMD, symbol Connector:TestPoint
- added U1: LMR36510ADDAR, Package_SO:Texas_HTSOP-8-1EP_3.9x4.9mm_P1.27mm_EP2.95x4.9mm_Mask2.4x3.1mm_ThermalVias, symbol Regulator_Switching:LMR36510ADDA
- added U2: TLV75533PDBVR, Package_TO_SOT_SMD:SOT-23-5, symbol Regulator_Linear:TLV75533PDBV
- added U3, U4: UCC12050DVER, footprints:DVE0016A, symbol UCC12050:UCC12050DVER
- added U5, U6: AMC0381D06QDFXRQ1, symbol precharge_custom:AMC0381D06QDFXRQ1
- added U7: STM32G031K8T6, Package_QFP:LQFP-32_7x7mm_P0.8mm, symbol MCU_ST_STM32G0:STM32G031K8Tx
- added U8: UCC27524AQDRQ1, Package_SO:SOIC-8_3.9x4.9mm_P1.27mm, symbol precharge_drivers:UCC27524AQDRQ1
Connections:
- new net: Q1.1 (G), R4.2, R7.1
- new net: D9.2 (A), R13.1
- new net: C1.1, D1.1 (K), D2.1 (K), R1.2
- new net: D1.2 (A), F1.1
- new net: F1.2, J1.1 (Pin_1)
- new net: C2.1, R1.1, U1.2 (VIN), U1.3 (EN)
- new net: J3.1 (Pin_1), U6.1 (HVIN)
- new net: C21.1, U6.4 (SNSP)
- new net: D7.2 (A), R11.1
- new net: D6.2 (A), R10.1
- new net: J2.1 (Pin_1), U5.1 (HVIN)
- new net: R2.1, R3.2, U1.5 (FB)
- new net: C4.1, U1.7 (BOOT)
- new net: C4.2, L1.2, U1.8 (SW)
- new net: D8.2 (A), R12.1
- new net: Q2.1 (G), R5.2, R8.1
- new net: C3.1, U1.6 (VCC)
- new net: C18.1, U5.4 (SNSP)
- new net: Q3.1 (G), R9.1
- new net +3V3: C19.1, C22.1, C23.1, C24.1, C27.1, C29.1, C8.2, J5.1 (Pin_1), R13.2, TP2.1, U2.5 (OUT), U5.14 (VDD2), U6.14 (VDD2), U7.4 (VDD)
- new net +5V: C10.2, C13.2, C14.2, C30.1, C31.1, C5.1, C6.2, C7.2, C9.2, L1.1, R2.2, TP3.1, U2.1 (IN), U2.3 (EN), U3.1 (EN), U3.3 (VINP), U4.1 (EN), U4.3 (VINP), U8.6 (VDD)
- new net CTRL_ENABLE: R6.2, R9.2, U7.17 (PB2)
- new net CTRL_ENABLE_SW: D5.2 (A), J7.2 (Pin_2), Q3.3 (D)
- new net DC_ISO_5V: C15.2, C16.2, C20.1, C28.1, U4.13 (SEL), U4.14 (VISO), U6.5 (VDD1)
- new net DC_ISO_GND: C15.1, C16.1, C20.2, C21.2, C28.2, J3.2 (Pin_2), U4.10 (NCS), U4.11 (NCS), U4.12 (NCS), U4.15 (GNDS), U4.16 (GNDS), U4.9 (GNDS), U6.2 (SNSN), U6.6 (GND1)
- new net DC_OUTN: U6.10 (OUTN), U7.10 (PA3)
- new net DC_OUTP: TP6.1, U6.11 (OUTP), U7.9 (PA2)
- new net GND: C1.2, C10.1, C13.1, C14.1, C19.2, C2.2, C22.2, C23.2, C24.2, C25.2, C27.2, C29.2, C3.2, C30.2, C31.2, C5.2, C6.1, C7.1, C8.1, C9.1, D2.2 (A), D6.1 (K), D7.1 (K), D8.1 (K), D9.1 (K), J1.2 (Pin_2), J5.5 (Pin_5), J8.2 (Pin_2), Q1.3 (S), Q2.3 (S), Q3.2 (S), R14.2, R15.2, R16.2, R17.2, R3.1, R4.1, R5.1, R6.1, TP4.1, U1.1 (PGND), U1.9 (PAD), U2.2 (GND), U3.2 (GNDP), U3.4 (SYNC), U3.6 (NCP), U3.7 (NCP), U3.8 (NCP), U4.2 (GNDP), U4.4 (SYNC), U4.6 (NCP), U4.7 (NCP), U4.8 (NCP), U5.9 (GND2), U6.9 (GND2), U7.5 (VSS), U8.3 (GND)
- new net LED_GREEN_CMD: R10.2, U7.11 (PA4)
- new net LED_RED_CMD: R12.2, U7.13 (PA6)
- new net LED_YELLOW_CMD: R11.2, U7.12 (PA5)
- new net MAIN_CMD: R15.1, TP8.1, U7.16 (PB1), U8.4 (INB)
- new net MAIN_GATE_DRIVE: R8.2, U8.5 (OUTB)
- new net MAIN_PERMIT_TBD: R17.1, U8.8 (ENB)
- new net MAIN_SW: D4.2 (A), J6.2 (Pin_2), Q2.2 (D)
- new net NRST: C25.1, J5.4 (Pin_4), U7.6 (PF2)
- new net PACK_ISO_5V: C11.2, C12.2, C17.1, C26.1, U3.13 (SEL), U3.14 (VISO), U5.5 (VDD1)
- new net PACK_ISO_GND: C11.1, C12.1, C17.2, C18.2, C26.2, J2.2 (Pin_2), U3.10 (NCS), U3.11 (NCS), U3.12 (NCS), U3.15 (GNDS), U3.16 (GNDS), U3.9 (GNDS), U5.2 (SNSN), U5.6 (GND1)
- new net PACK_OUTN: U5.10 (OUTN), U7.8 (PA1)
- new net PACK_OUTP: TP5.1, U5.11 (OUTP), U7.7 (PA0)
- new net PRECHARGE_CMD: R14.1, TP7.1, U7.15 (PB0), U8.2 (INA)
- new net PRECHARGE_SW: D3.2 (A2), J4.2 (Pin_2), Q1.2 (D)
- new net PRE_GATE_DRIVE: R7.2, U8.7 (OUTA)
- new net PRE_PERMIT_TBD: R16.1, U8.1 (ENA)
- new net SDC_12V_COIL: D3.1 (A1), D4.1 (K), D5.1 (K), J4.1 (Pin_1), J6.1 (Pin_1), J7.1 (Pin_1), J8.1 (Pin_1), TP1.1
- new net SWCLK: J5.3 (Pin_3), U7.25 (PA14)
- new net SWDIO: J5.2 (Pin_2), U7.24 (PA13)
- no-connect marks 0 -> 18
Other:
- note added: "01 GLV INPUT / PROTECTION"
- note added: "02 12V TO 5V / 1A BUCK"
- note added: "03 5V TO 3V3"
- note added: "04 EXTERNAL SDC COIL POWER"
- note added: "05 PACK / ISOLATED VOLTAGE SENSING"
- note added: "06 DC-LINK / ISOLATED VOLTAGE SENSING"
- note added: "07 MCU / ADC / CONTROL"
- note added: "08 GATE DRIVE / PERMITS TBD"
- note added: "09 PRECHARGE / P105BDA"
- note added: "1 = downstream SDC +12V 2 = GLV return"
- note added: "10 MAIN AIR / EV200 CANDIDATE"
- note added: "11 STATUS INDICATION"
- note added: "12 GLV TEST POINTS / MEASUREMENTS"
- note added: "13 RESERVED OUTPUT / DNP"
- note added: "1=SDC +12V 2=switched return"
- note added: "Future use only; CTRL_ENABLE function not finalized."
- note added: "GLV ADC"
- note added: "ISOLATED HV"
- note added: "No permit source fitted: outputs default DISABLED. Resolve SDC-state / re-arm / AIR interlocks before PCB release."
- note added: "SDC must directly interrupt AIR / precharge coil current. External source only; do not bridge to J1 logic input."
- note added: "SWD: 1=3V3 2=SWDIO 3=SWCLK 4=NRST 5=GND"
- company: (none) -> Sun Devil Motorsports
- title: (none) -> SDM EV - Standalone Precharge Controller
